Commit message: neater urdf and launch file

File: urdf/2link_robot.urdf (robot description, URDF)
Before this commit: robot 2link_robot, 2 links, 1 joints
Links:
- added link pseudo_link
- link base_link: geometry visual box size=0.7 .05 .05
- link second_link: geometry visual box size=0.7 .05 .05
Joints:
- added joint ee: type fixed, parent second_link, child pseudo_link, origin xyz=0.7 0 0 rpy=0 0 0
- joint joint1: origin xyz=0.6 0 0 rpy=0 0 0 -> xyz=0.7 0 0 rpy=0 0 0

Commit message: actually neater urdf and launch file

File: urdf/2link_robot.urdf (robot description, URDF)
Before this commit: robot 2link_robot, 3 links, 2 joints
Links:
- removed link base_link
- removed link pseudo_link
- removed link second_link
- added link arm1; visual box size=1 .05 .05
- added link arm2; visual box size=1 .05 .05
- added link base
- added link endEffector
Joints:
- removed joint ee
- removed joint joint1
- added joint baseHinge: type continuous, parent base, child arm1, axis 0 0 1
- added joint ee_frame: type fixed, parent arm2, child endEffector, origin xyz=1 0 0 rpy=0 0 0
- added joint interArm: type continuous, parent arm1, child arm2, origin xyz=1 0 0 rpy=0 0 0, axis 0 0 1

Commit message: finally moving as it should

File: urdf/2link_robot.urdf (robot description, URDF)
Before this commit: robot 2link_robot, 4 links, 3 joints
Joints:
- removed joint ee_frame
- added joint ee_joint: type fixed, parent arm2, child endEffector, origin xyz=1 0 0 rpy=0 0 0
